File: nand/board/board/board.kicad_pcb (KiCad board)
At the start: 2 copper layers, 74.9 x 59.7 mm, 40 parts, among them J1 Conn_01x13, J2 SWD1, J3 gnd, J4 SWD3, J5 3v3, J6 SWD2, J7 Raspberry_Pi_2_3, SW1 PTS645SJH73LFS, SW2 PTS645SJH73LFS, SW3 PTS645SJH73LFS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

Commit message: ... hours later ...
Parts:
- moved C15 2.17 mm to (137.7, 132.6)
Routing:
- net Net-(U1-Pad36): track 0.00 -> 109.0 mm, vias 0 -> 6
- net Net-(U1-Pad33): track 0.00 -> 95.7 mm, vias 0 -> 6
- net Net-(U1-Pad35): track 0.00 -> 93.3 mm, vias 0 -> 6
- net Net-(U1-Pad34): track 0.00 -> 90.7 mm, vias 0 -> 6
- net Net-(J1-Pad1): track 0.00 -> 79.5 mm, vias 0 -> 4
- net Net-(U1-Pad30): track 0.00 -> 76.8 mm, vias 0 -> 2
- net Net-(U1-Pad27): track 0.00 -> 72.5 mm, vias 0 -> 2
- net NRST3: track 16.3 -> 85.2 mm, vias 0 -> 4
- net e1: track 0.00 -> 69.0 mm, vias 0 -> 6
- net Net-(U1-Pad29): track 0.00 -> 66.6 mm, vias 0 -> 2
- net SWCLK1: track 0.00 -> 66.3 mm, vias 0 -> 5
- net a0: track 0.00 -> 66.3 mm, vias 0 -> 2
- net NRST1: track 18.2 -> 83.6 mm, vias 0 -> 3
- net SWDIO1: track 0.00 -> 64.6 mm, vias 0 -> 4
- net Net-(U1-Pad23): track 0.00 -> 63.3 mm, vias 0 -> 2
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Other:
- board size 74.9 x 59.7 mm -> 76.2 x 59.7 mm

Commit message: v1 board sent for manufacturing
Routing:
- net Net-(J6-Pad2): track 0.00 -> 58.4 mm, vias 0 -> 2
- net BOOT2: track 0.00 -> 57.6 mm, vias 0 -> 2
- net 3v3: track 520.4 -> 567.9 mm
- net GND: track 631.1 -> 640.5 mm
- net Net-(U3-Pad2): track 26.1 -> 35.1 mm
- net NRST3: track 85.2 -> 81.4 mm
- net e1: track 69.0 -> 65.5 mm
- net Net-(U1-Pad33): track 95.7 -> 97.6 mm
- net BOOT3: track 51.6 -> 52.8 mm
- net Net-(U3-Pad37): track 18.2 -> 19.3 mm
- net i2: track 25.3 -> 24.2 mm
- net Net-(J1-Pad5): track 41.4 -> 40.2 mm
- net Net-(C4-Pad2): track 16.5 -> 15.5 mm
- net Net-(U3-Pad36): track 27.2 -> 28.2 mm
- net Net-(U1-Pad29): track 66.6 -> 65.7 mm
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- added copper zone on F.Cu, net 3v3
- added copper zone on B.Cu, net GND
Other:
- board size 76.2 x 59.7 mm -> 76.2 x 58.4 mm
- board text added: "@tom7"
- board text added: "META FPU"
- board text added: "v1"
