File: nand/board/board/board.sch (KiCad schematic (older format))
At the start: 40 parts, among them J1 Conn_01x13, J2 SWD1, J3 gnd, J4 SWD3, J5 3v3, J6 SWD2, J7 Raspberry_Pi_2_3, SW1 PTS645SJH73LFS, SW2 PTS645SJH73LFS, SW3 PTS645SJH73LFS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

Commit message: v1 board sent for manufacturing
Changed lines of the file:
@@
 EESchema Schematic File Version 4
+LIBS:board-cache
 EELAYER 26 0
 EELAYER END
@@
 Wire Wire Line
 	4150 2250 4300 2250
-Connection ~ 4450 2900
-Wire Wire Line
-	4450 2900 4500 2900
-Connection ~ 4450 3000
-Wire Wire Line
-	4450 3000 4500 3000
 $Comp
 L boardparts:PTS645SJH73LFS SW1
