File: pingu/board/testboard/stackboard/stackboard.kicad_pcb (KiCad board)
At the start: 2 copper layers, 161.3 x 91.4 mm, 65 parts, among them J1 Raspberry_Pi_2_3, J2 board sel, J3 Group Sel A, J4 Group Sel B, J5 common up, J6 Board Sel, J7 Group Sel, J8 common down, Q1 2N3904, Q2 2N3904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

Commit message: Stackboard sent for manufacturing
Parts:
- removed SDA6: SDA6, Connector_PinHeader_2.54mm:PinHeader_1x01_P2.54mm_Vertical
- added EN0: EN0, Connector_PinHeader_2.54mm:PinHeader_1x01_P2.54mm_Vertical, F.Cu at (66.0, 38.7)
- added G***: LOGO, myfeets:logo, F.Cu at (117.5, 55.9)
- added J10: com alt, Connector_PinHeader_2.54mm:PinHeader_1x07_P2.54mm_Vertical, F.Cu at (54.6, 97.8)
- added J9: Up, Connector_PinHeader_2.54mm:PinHeader_1x01_P2.54mm_Vertical, F.Cu at (66.7, 97.8)
- added REF**: MountingHole_2.5mm, MountingHole:MountingHole_2.5mm, F.Cu at (15.9, 15.2)
- added REF**: MountingHole_2.5mm, MountingHole:MountingHole_2.5mm, F.Cu at (25.4, 80.6)
- added SCL1: SCL1, Connector_PinHeader_2.54mm:PinHeader_1x01_P2.54mm_Vertical, F.Cu at (117.5, 36.8)
- added SDA0: SDA0, Connector_PinHeader_2.54mm:PinHeader_1x01_P2.54mm_Vertical, F.Cu at (72.4, 38.1)
- added SDA1: SDA1, Connector_PinHeader_2.54mm:PinHeader_1x01_P2.54mm_Vertical, F.Cu at (117.5, 33.0)
- added TP10: GND, Connector_PinHeader_2.54mm:PinHeader_1x01_P2.54mm_Vertical, F.Cu at (122.6, 93.3)
- added TP11: 3v3, Connector_PinHeader_2.54mm:PinHeader_1x01_P2.54mm_Vertical, F.Cu at (170.2, 57.1)
- added TP12: GND, Connector_PinHeader_2.54mm:PinHeader_1x01_P2.54mm_Vertical, F.Cu at (29.2, 15.9)
- added TP19: 19, Connector_PinHeader_2.54mm:PinHeader_1x01_P2.54mm_Vertical, F.Cu at (25.4, 87.0)
- added TP4: 5v, Connector_PinHeader_2.54mm:PinHeader_1x01_P2.54mm_Vertical, F.Cu at (23.5, 49.5)
- added TP6: SCL, Connector_PinHeader_2.54mm:PinHeader_1x01_P2.54mm_Vertical, F.Cu at (71.8, 43.2)
- added TP7: 3v3, Connector_PinHeader_2.54mm:PinHeader_1x01_P2.54mm_Vertical, F.Cu at (121.9, 16.5)
- added TP8: GND, Connector_PinHeader_2.54mm:PinHeader_1x01_P2.54mm_Vertical, F.Cu at (63.5, 54.6)
- moved R2 132.1 mm to (40.0, 21.0)
- moved R6 130.3 mm to (40.0, 31.1)
- moved R10 120.3 mm to (40.0, 33.7)
- moved R18 119.3 mm to (66.7, 74.9)
- moved R14 114.5 mm to (40.0, 50.8)
- moved R17 114.3 mm to (40.0, 58.4)
- moved R1 112.4 mm to (40.0, 18.4)
- moved R21 108.7 mm to (59.1, 71.1), turned to 180 degrees
- moved R11 105.0 mm to (40.0, 43.2)
- moved R16 102.7 mm to (40.0, 55.9)
- moved R3 101.4 mm to (40.0, 23.5)
- moved R12 100.0 mm to (40.0, 45.7)
- moved R4 98.6 mm to (40.0, 26.0)
- moved R15 98.3 mm to (40.0, 53.3)
- moved R5 98.1 mm to (40.0, 28.6), turned to 0 degrees
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- renumbered J1 to pi
Routing:
- net 3v3: track 67.6 -> 271.3 mm, vias 0 -> 7
- net Net-(EN0-Pad1): track 9.82 -> 116.4 mm, vias 2 -> 4
- net Net-(R3-Pad1): track 6.61 -> 110.2 mm, vias 0 -> 4
- net SCL: track 236.1 -> 334.7 mm, vias 12 -> 13
- net Net-(R5-Pad1): track 65.5 -> 163.2 mm, vias 3 -> 4
- net Net-(R10-Pad1): track 63.9 -> 161.0 mm, vias 3 -> 7
- net Net-(J1-Pad11): track 0.00 -> 88.9 mm, vias 0 -> 1
- net SDA: track 236.8 -> 323.0 mm, vias 9 -> 10
- net Net-(R13-Pad1): track 8.28 -> 90.8 mm, vias 0 -> 2
- net a4: track 0.00 -> 75.0 mm, vias 0 -> 1
- net Net-(R11-Pad1): track 6.17 -> 80.3 mm, vias 2 -> 3
- net Net-(LED4-Pad1): track 0.00 -> 70.3 mm, vias 0 -> 3
- net GND: track 92.9 -> 158.9 mm
- net a0: track 13.2 -> 78.2 mm, vias 0 -> 1
- net a3: track 0.00 -> 58.8 mm, vias 0 -> 2
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Other:
- board size 161.3 x 91.4 mm -> 161.9 x 91.4 mm
- board text added: "(fanout)"
- board text added: "10k"
